File: GD.kicad_sch (KiCad schematic)
At the start: 18 parts, among them U4 TMV 0512SHI, U5 UCC5304DWVR

Commit message: Add files via upload
Parts:
- removed D8, D9: LED_ABGR, LED_SMD:LED_0805_2012Metric, symbol Device:LED_ABGR
- added D5, D7: SMLMN2WB1CW1, LED_SMD:LED_0805_2012Metric, symbol Device:LED
- C10, C12: Part No. TMCP1E105MTRF -> TAJP106M010RNJ
- C11: Part No. TMCP1E105MTRF -> 298D227X0004P2T
- C6, C7, C8: Part No. TMCP1E105MTRF -> T58W9105M035C0500
- C9: value C -> 33p; Part No. (none) -> 600F330FT250XT4K
- D6: Part No. (none) -> US2AA
- R9: value R -> 51; Part No. (none) -> RC0805FR-0751RL
Connections:
- net ISO_12: now also D5.2 (A)
- net VG: now also D7.2 (A)
- net at R13.1: now also D7.1 (K)
- net at R5.1: now also D5.1 (K)
