File: LPF.kicad_sch (KiCad schematic)
At the start: 7 parts, among them U3 OPA547T

Commit message: Add files via upload
Parts:
- removed U3: OPA547T, OPA547Tfootprints:KVT7, symbol 2025-02-25_02-40-25:OPA547T
- added U1: LM358AP, LM358AP_footprints:P8, symbol 2025-03-01_21-15-45:LM358AP
- C2: Part No. TMCP1E105MTRF -> T58W9105M035C0500
Connections:
- net +3.3V: now also U1.8 (VCC)
- net GND: now also U1.4 (GND)
- net OUT: now also R2.2, U1.1 (1OUT)
- net at C1.1, R3.2, R4.2: now also U1.3 (1IN+)
- net at R1.2, R2.1: now also U1.2 (1IN-)
- no-connect marks 0 -> 3
Other:
- moved on the sheet: C1, C2, R1, R2, R3, R4
