File: MCU.kicad_sch (KiCad schematic)
At the start: 7 parts, among them U2 LAUNCHXL-F28379D

Commit message: Add files via upload
Parts:
- removed D10, D11, D12: LED_ABGR, LED_SMD:LED_0805_2012Metric, symbol Device:LED_ABGR
- added D2, D3, D4: LTST-C171GKT, LED_SMD:LED_0805_2012Metric, symbol Device:LED
- U2: Part No. (none) -> LAUNCHXL-F28379D
Connections:
- net +3.3V: now also D3.2 (A)
- net +5V: now also D2.2 (A)
- net PWM: now also D4.2 (A)
- net at R7.1: now also D3.1 (K)
- net at R8.1: now also D4.1 (K)
- net at R6.1: now also D2.1 (K)
- net VFILTD renamed VFILT
- no-connect marks 89 -> 88
Other:
- moved on the sheet: R6, R7, R8, U2E
