File: PCB_Tutorial_Lect.kicad_pcb (KiCad board)
At the start: 2 copper layers, 132.5 x 137.5 mm, 43 parts, among them J1 Conn_01x01_Pin, J2 Conn_01x01_Pin, J3 Conn_01x01_Pin, J4 Conn_01x01_Pin, J5 Conn_01x01_Pin, Q1 IRF540N, U2 LAUNCHXL-F28379D, U3 OPA547T, U4 TMV 0512SHI, U5 UCC5304DWVR

Commit message: Add files via upload
Parts:
- removed D10, D11, D12, D8, D9: LED_ABGR, LED_SMD:LED_0805_2012Metric
- removed U3: OPA547T, OPA547Tfootprints:KVT7
- added D2: LTST-C171GKT, LED_SMD:LED_0805_2012Metric, F.Cu at (80.0, 99.0)
- added D3: LTST-C171GKT, LED_SMD:LED_0805_2012Metric, F.Cu at (170.0, 98.0)
- added D4: LTST-C171GKT, LED_SMD:LED_0805_2012Metric, F.Cu at (50.1, 85.0)
- added D5: SMLMN2WB1CW1, LED_SMD:LED_0805_2012Metric, F.Cu at (61.9, 88.5)
- added D7: SMLMN2WB1CW1, LED_SMD:LED_0805_2012Metric, F.Cu at (78.0, 67.0)
- added G***: LOGO, UWINLOGO:UWINLOGO.pretty, F.Cu at (66.0, 162.5)
- added G***: LOGO, MURATAPSLOGO:murataPSlogo.pretty, F.Cu at (148.5, 164.5)
- added H1: MountingHole, MountingHole:MountingHole_4mm, F.Cu at (51.5, 32.5)
- added H2: MountingHole, MountingHole:MountingHole_4mm, F.Cu at (167.0, 32.5)
- added H3: MountingHole, MountingHole:MountingHole_4mm, F.Cu at (52.5, 164.5)
- added H4: MountingHole, MountingHole:MountingHole_4mm, F.Cu at (167.5, 164.5)
- added U1: LM358AP, LM358AP_footprints:P8, F.Cu at (157.0, 86.5)
- C5: value ? -> 47uf
- C9: value C -> 33p
- L1: value ? -> 47mh; footprint Inductor_THT:L_Radial_D50.8mm_P38.86mm_Vishay_IHB-6 -> 5500R_566Kfootprints:5500R-566K_API
- R9: value R -> 51
- moved J3 48.1 mm to (121.0, 43.5)
- moved J2 47.6 mm to (121.5, 56.5)
- moved L1 23.7 mm to (127.0, 88.5)
Connections:
- R2 pad 2: Net-(U3-VIN-) -> /VFILT
- U2 pad J3_3: /VFILTD -> /VFILT
Routing:
- net /VFILT: track 0.00 -> 55.0 mm, vias 0 -> 1
- net /VOUT: track 82.0 -> 109.8 mm
- net /VSW: track 141.0 -> 160.8 mm
- net GND: track 16.9 -> 31.0 mm, vias 2 -> 5
- net Net-(U3-VIN-): track 13.2 -> 0.00 mm, vias 2 -> 0
- net Net-(U1-1IN+): track 20.5 -> 8.82 mm
- net +3.3V: track 42.8 -> 37.9 mm
- net Net-(U1-1IN-): track 3.43 -> 5.55 mm
Other:
- board size 132.5 x 137.5 mm -> 132.5 x 142 mm
- board text added: "5500R-566K"
- board text added: "GND"
- board text added: "LM358AP"
- board text added: "VIN"
- board text added: "VOUT"
- board text added: "VSW"
- board text added: "WINTER 2025: GROUP 10 Abdullah Zafar Conor St. Andrews Trevor Dyck"
