File: PCB_Tutorial_Lect.kicad_sch (KiCad schematic)
At the start: 0 parts

Commit message: Add files via upload
Parts:
- added H1, H2, H3, H4: MountingHole, MountingHole:MountingHole_4mm, symbol Mechanical:MountingHole
Other:
- sheet MCU ports: added VFILT; removed VFILTD
